File: Panel_PCB/Panel_PCB.kicad_pcb (KiCad board)
At the start: 2 copper layers, 140 parts, among them J1 Relay 1, J1 Screw_Terminal_01x20, J16 Boton 2, J17 Boton 3, J18 Sensor IN sgn, J19 Sensor OUT sgn, J2 Relay 2, J2 Screw_Terminal_01x20, J20 Boton 1, J21 Boton 1 sgn, J22 Sensor IN, J23 Sensor OUT, J24 Boton 2 sgn, J25 Boton 3 sgn, J3 Relay 3, J3 Screw_Terminal_01x20, J4 Relay 4, J4 Screw_Terminal_01x20, J5 AC, J6 Bateria, J7 AC, J8 AC, K1 SANYOU_SRD_Form_C, K14 SANYOU_SRD_Form_C, K2 SANYOU_SRD_Form_C, K4 EC2-4.5SNU, K8 SANYOU_SRD_Form_C, K9 SANYOU_SRD_Form_C, Q1 2N2222A, Q1 Q_NPN, Q2 2N2222A, Q2 Q_NPN, Q3 2N2222A, Q3 Q_NPN, Q4 Q_NPN, Q5 2N2222A, T1 Transformer_1P_1S, U1 4N35, U1 TLP291, U15 LM7805_TO220, U16 LM1117T-3.3, U2 ESP32-WROOM-32, U2 TLP291, U20 LM1117T-3.3, U21 LM7812_TO220, U3 CH340C, U3 TLP291, U4 LM1117T-3.3, U4 LM7805_TO220, U5 TLP291, U6 LM7812_TO220

Commit message: Organizando elementos del PCB
Parts:
- removed 3v3_2, gnd1_2, gpio15_2, gpio16_2, gpio17_2, gpio18_2, gpio19_2, gpio1_2, gpio21_2, gpio22_2, gpio23_2, gpio2_2, gpio3_2, gpio4_2, gpio5_2, pin_x1, pin_x10, pin_x2, pin_x3, pin_x4, pin_x5, pin_x6, pin_x7, pin_x8, pin_x9: ~, Connector_Wire:SolderWire-0.75sqmm_1x01_D1.25mm_OD2.3mm
- removed the J1 at (1.62, 32.0)
- removed the J1 at (126.6, 0.70)
- removed J19: Sensor OUT sgn, TerminalBlock_Phoenix:TerminalBlock_Phoenix_MKDS-1,5-2-5.08_1x02_P5.08mm_Horizontal
- removed the J2 at (1.62, 44.1)
- removed the J2 at (156.6, 48.7)
- removed J20: Boton 1, TerminalBlock_Phoenix:TerminalBlock_Phoenix_MKDS-1,5-2-5.08_1x02_P5.08mm_Horizontal
- removed J21: Boton 1 sgn, TerminalBlock_Phoenix:TerminalBlock_Phoenix_MKDS-1,5-2-5.08_1x02_P5.08mm_Horizontal
- removed J22: Sensor IN, TerminalBlock_Phoenix:TerminalBlock_Phoenix_MKDS-1,5-2-5.08_1x02_P5.08mm_Horizontal
- removed J23: Sensor OUT, TerminalBlock_Phoenix:TerminalBlock_Phoenix_MKDS-1,5-2-5.08_1x02_P5.08mm_Horizontal
- removed J24: Boton 2 sgn, TerminalBlock_Phoenix:TerminalBlock_Phoenix_MKDS-1,5-2-5.08_1x02_P5.08mm_Horizontal
- removed J25: Boton 3 sgn, TerminalBlock_Phoenix:TerminalBlock_Phoenix_MKDS-1,5-2-5.08_1x02_P5.08mm_Horizontal
- removed the J3 at (1.62, 56.3)
- removed the J3 at (55.0, 40.5)
- removed the J4 at (1.62, 68.4)
- removed the J4 at (24.9, -7.80)
- removed the K1 at (-134.8, -25.3)
- removed the K1 at (255.6, 138.7)
- removed K14, K8, K9: SANYOU_SRD_Form_C, Relay_THT:Relay_SPDT_SANYOU_SRD_Series_Form_C
- removed the Q1 at (204.2, 44.4)
- removed the Q1 at (31.6, 177.4)
- removed the Q2 at (31.6, 183.2)
- removed the Q2 at (204.2, 50.1)
- removed the Q3 at (31.6, 189.0)
- removed the Q3 at (204.2, 55.9)
- removed Q5: 2N2222A, Package_TO_SOT_THT:TO-92
- removed T1: Transformer_1P_1S, Transformer_THT:Transformer_NF_ETAL_1-1_P1200
- removed the U1 at (229.6, 46.1)
- removed the U1 at (-84.8, 35.0)
- removed U15: LM7805_TO220, Package_TO_SOT_THT:TO-220-3_Vertical
- removed U16, U20: LM1117T-3.3, Package_TO_SOT_THT:TO-220-3_Horizontal_TabDown
- removed the U2 at (251.8, -2.36)
- removed the U2 at (-84.8, 39.1)
- removed U21: LM7812_TO220, Package_TO_SOT_THT:TO-220-3_Vertical
- removed the U3 at (237.7, 100.4)
- removed the U3 at (-84.8, 43.3)
- removed the U4 at (127.3, 117.2)
- removed the U4 at (-92.9, 17.3)
- added J1: AC, TerminalBlock_Phoenix:TerminalBlock_Phoenix_MKDS-1,5-2-5.08_1x02_P5.08mm_Horizontal, F.Cu at (-114.2, 97.9)
- added J10: Relay 3, TerminalBlock_Phoenix:TerminalBlock_Phoenix_MKDS-1,5-2-5.08_1x02_P5.08mm_Horizontal, F.Cu at (606.3, 329.2)
- added J11: Relay 4, TerminalBlock_Phoenix:TerminalBlock_Phoenix_MKDS-1,5-2-5.08_1x02_P5.08mm_Horizontal, F.Cu at (719.0, 331.6)
- added J12: AC, TerminalBlock_Phoenix:TerminalBlock_Phoenix_MKDS-1,5-2-5.08_1x02_P5.08mm_Horizontal, F.Cu at (-48.8, 92.8)
- added J13: AC, TerminalBlock_Phoenix:TerminalBlock_Phoenix_MKDS-1,5-2-5.08_1x02_P5.08mm_Horizontal, F.Cu at (-9.46, 97.8)
- added J14: Sensor IN sgn, TerminalBlock_Phoenix:TerminalBlock_Phoenix_MKDS-1,5-2-5.08_1x02_P5.08mm_Horizontal, F.Cu at (681.4, -51.7)
- added J15: Sensor OUT sgn, TerminalBlock_Phoenix:TerminalBlock_Phoenix_MKDS-1,5-2-5.08_1x02_P5.08mm_Horizontal, F.Cu at (681.6, -28.8)
- added J2: Bateria, TerminalBlock_Phoenix:TerminalBlock_Phoenix_MKDS-1,5-2-5.08_1x02_P5.08mm_Horizontal, F.Cu at (277.7, 12.8)
- added J3: Sensor IN, TerminalBlock_Phoenix:TerminalBlock_Phoenix_MKDS-1,5-2-5.08_1x02_P5.08mm_Horizontal, F.Cu at (391.6, -7.93)
- added J4: Sensor OUT, TerminalBlock_Phoenix:TerminalBlock_Phoenix_MKDS-1,5-2-5.08_1x02_P5.08mm_Horizontal, F.Cu at (418.9, -7.80)
- added J9: Relay 2, TerminalBlock_Phoenix:TerminalBlock_Phoenix_MKDS-1,5-2-5.08_1x02_P5.08mm_Horizontal, F.Cu at (503.9, 344.7)
- added K1: SANYOU_SRD_Form_C, Relay_THT:Relay_SPDT_SANYOU_SRD_Series_Form_C, F.Cu at (394.7, 281.7)
- added K3: SANYOU_SRD_Form_C, Relay_THT:Relay_SPDT_SANYOU_SRD_Series_Form_C, F.Cu at (598.0, 283.0)
- added K5: EC2-4.5SNU, Relay_THT:Relay_DPDT_Kemet_EC2_NU, F.Cu at (-19.4, 60.3)
- added K6: SANYOU_SRD_Form_C, Relay_THT:Relay_SPDT_SANYOU_SRD_Series_Form_C, F.Cu at (139.2, 140.7)
- added Q1: 2N2222A, Package_TO_SOT_THT:TO-92, F.Cu at (400.1, 255.7)
- added Q2: 2N2222A, Package_TO_SOT_THT:TO-92, F.Cu at (500.5, 259.9)
- added Q3: 2N2222A, Package_TO_SOT_THT:TO-92, F.Cu at (595.8, 258.1)
- added U1: TLP291, Package_SO:SOIC-4_4.55x2.6mm_P1.27mm, F.Cu at (402.5, 237.9)
- added U10: LM1117T-3.3, Package_TO_SOT_THT:TO-220-3_Horizontal_TabDown, F.Cu at (456.8, 102.7)
- added U2: TLP291, Package_SO:SOIC-4_4.55x2.6mm_P1.27mm, F.Cu at (511.0, 246.6)
- added U3: TLP291, Package_SO:SOIC-4_4.55x2.6mm_P1.27mm, F.Cu at (608.6, 245.9)
- added U4: TLP291, Package_SO:SOIC-4_4.55x2.6mm_P1.27mm, F.Cu at (719.2, 251.4)
- added U7: LM7805_TO220, Package_TO_SOT_THT:TO-220-3_Vertical, F.Cu at (379.9, 87.0)
- added U8: LM7805_TO220, Package_TO_SOT_THT:TO-220-3_Vertical, F.Cu at (382.1, 135.4)
- added U9: LM1117T-3.3, Package_TO_SOT_THT:TO-220-3_Horizontal_TabDown, F.Cu at (455.6, 59.5)
- C10, C8: value 100 μF -> 0.1 μF
- C11: value 10 μF -> 100 μF
- C12: value 0.22 μF -> 10 μF
- C13: value 0.1 μF -> 100 μF
- C14: value 35V 4700μF -> 10 μF; footprint Capacitor_THT:C_Radial_D18.0mm_H35.5mm_P7.50mm -> Capacitor_THT:C_Disc_D3.0mm_W1.6mm_P2.50mm
- C2: value 0.22 μF -> 35V 4700μF; footprint Capacitor_THT:C_Disc_D3.0mm_W1.6mm_P2.50mm -> Capacitor_THT:C_Radial_D18.0mm_H35.5mm_P7.50mm
- C3, C5, C7: value 0.1 μF -> 0.22 μF
- C4, C6: value 0.22 μF -> 0.1 μF
- C9: value 10 μF -> 0.22 μF
- J16: value Boton 2 -> Boton 1 sgn
- J17: value Boton 3 -> Boton 2 sgn
- J18: value Sensor IN sgn -> Boton 3 sgn
- J5: value AC -> Boton 1
- J6: value Bateria -> Boton 2
- J7: value AC -> Boton 3
- J8: value AC -> Relay 1
- K4: value EC2-4.5SNU -> SANYOU_SRD_Form_C; footprint Relay_THT:Relay_DPDT_Kemet_EC2_NU -> Relay_THT:Relay_SPDT_SANYOU_SRD_Series_Form_C
- Q4: value Q_NPN -> 2N2222A
- R3: value 450 -> 150
- R4: value R_US -> 450
- U5: value TLP291 -> LM7812_TO220; footprint Package_SO:SOIC-4_4.55x2.6mm_P1.27mm -> Package_TO_SOT_THT:TO-220-3_Vertical
- moved K4 844.6 mm to (710.7, 283.2)
- moved D6 826.7 mm to (689.6, 279.0), turned to -90 degrees
- moved GPIO25 745.1 mm to (629.2, 94.1)
- moved GPIO26 742.4 mm to (629.2, 98.8)
- moved GPIO27 742.4 mm to (629.2, 103.4)
- moved GPIO32 742.4 mm to (629.2, 108.1)
- moved GPIO34 741.0 mm to (634.0, 94.1)
- moved GPIO35 741.0 mm to (634.0, 98.8)
- moved GPIO33 740.0 mm to (629.2, 112.7)
- moved GPIO12 738.4 mm to (614.6, 112.7)
- moved GPIO36 738.4 mm to (634.0, 103.4)
- moved GPIO39 738.4 mm to (634.0, 108.1)
- moved VIN1 738.4 mm to (634.0, 112.7)
- moved GPIO13 736.9 mm to (619.5, 94.1)
- moved GPIO14 736.9 mm to (619.5, 98.8)
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Connections:
- C1 pad 1: Net-(D2-K) -> Net-(C1-Pad1)
- C10 pad 1: Net-(U16-VI) -> Net-(U8-VO)
- C11 pad 1: Net-(J18-Pin_1) -> Net-(U10-VI)
- C12 pad 1: Net-(D2-K) -> Net-(J14-Pin_1)
- C13 pad 1: Net-(D4-K) -> Net-(U10-VI)
- C14 pad 1: Net-(C14-Pad1) -> Net-(J16-Pin_1)
- C3 pad 1: Net-(U15-VI) -> Net-(D2-K)
- C4 pad 1: Net-(U15-VI) -> Net-(U5-VO)
- C5 pad 1: Net-(U15-VO) -> Net-(D2-K)
- C6 pad 1: Net-(U15-VI) -> Net-(D3-K)
- C7 pad 1: Net-(U16-VI) -> Net-(U5-VO)
- C8 pad 1: Net-(U16-VI) -> Net-(U10-VI)
- C9 pad 1: Net-(J21-Pin_1) -> Net-(U5-VO)
- D1 pad 3: Net-(J7-Pin_1) -> Net-(J13-Pin_1)
- D4 pad 1: Net-(D4-K) -> Net-(D3-K)
- D5 pad 1: Net-(D4-K) -> Net-(D3-K)
- D6 pad 1: Net-(D4-K) -> Net-(D3-K)
- D7 pad 1: Net-(D4-K) -> Net-(D7-K)
- F1 pad 1: Net-(J7-Pin_2) -> Net-(J1-Pin_2)
- F1 pad 2: Net-(D1-Pad2) -> Net-(J12-Pin_1)
- F2 pad 1: Net-(J5-Pin_2) -> Net-(J13-Pin_2)
- F2 pad 2: Net-(J8-Pin_1) -> Net-(D1-Pad2)
- J16 pad 1: Net-(D1--) -> Net-(J16-Pin_1)
- J17 pad 1: Net-(D1--) -> Net-(J16-Pin_1)
- J18 pad 1: Net-(J18-Pin_1) -> Net-(J16-Pin_1)
- J5 pad 1: Net-(J5-Pin_1) -> Net-(D1--)
- J5 pad 2: Net-(J5-Pin_2) -> Net-(J16-Pin_2)
- J6 pad 1: Net-(D3-A) -> Net-(D1--)
- J6 pad 2: Net-(D1--) -> Net-(J17-Pin_2)
- J7 pad 1: Net-(J7-Pin_1) -> Net-(D1--)
- J7 pad 2: Net-(J7-Pin_2) -> Net-(J18-Pin_2)
- J8 pad 2: Net-(J5-Pin_1) -> Net-(J8-Pin_2)
- K2 pad 2: Net-(D7-A) -> Net-(D4-A)
- K2 pad 5: Net-(D4-K) -> Net-(D3-K)
- K4 pad 1: Net-(J8-Pin_1) -> Net-(J11-Pin_2)
- K4 pad 3: unconnected-(K4-Pad3) -> Net-(J11-Pin_1)
- K4 pad 4: Net-(C14-Pad1) -> unconnected-(K4-Pad4)
- K4 pad 5: Net-(K4-Pad5) -> Net-(D3-K)
- Q4 pad 1: (no net) -> Net-(Q4-E)
- Q4 pad 2: (no net) -> Net-(Q4-B)
- Q4 pad 3: (no net) -> Net-(D6-A)
- R1 pad 2: Net-(C14-Pad1) -> Net-(C1-Pad1)
- R10 pad 1: Net-(D4-K) -> Net-(D3-K)
- R2 pad 1: Net-(K4-Pad5) -> Net-(K5-Pad5)
- R3 pad 1: Net-(D4-K) -> Net-(Q1-E)
- R3 pad 2: Net-(R3-Pad2) -> Net-(D1--)
- R4 pad 1: Net-(Q5-E) -> Net-(D3-K)
- R4 pad 2: Net-(D1--) -> Net-(R4-Pad2)
- R6 pad 1: Net-(D4-K) -> Net-(D3-K)
- R8 pad 1: Net-(D4-K) -> Net-(D3-K)
- R9 pad 1: Net-(Q3-E) (its old number) -> Net-(Q4-E)
- U5 pad 1: unconnected-(U5-Pad1) -> Net-(D2-K)
- U5 pad 3: Net-(Q3-B) -> Net-(U5-VO)
- U6 pad 3: Net-(U15-VI) -> Net-(D3-K)
- VIN1 pad 1: Net-(U15-VO) -> Net-(U8-VO)
Other:
- board text removed: "Bojtronic"
- board text removed: "Security Software"

Commit message: Conexiones al microcontrolador
Parts:
- removed J14: Sensor IN sgn, TerminalBlock_Phoenix:TerminalBlock_Phoenix_MKDS-1,5-2-5.08_1x02_P5.08mm_Horizontal
- removed J15: Sensor OUT sgn, TerminalBlock_Phoenix:TerminalBlock_Phoenix_MKDS-1,5-2-5.08_1x02_P5.08mm_Horizontal
- removed J16: Boton 1 sgn, TerminalBlock_Phoenix:TerminalBlock_Phoenix_MKDS-1,5-2-5.08_1x02_P5.08mm_Horizontal
- removed J17: Boton 2 sgn, TerminalBlock_Phoenix:TerminalBlock_Phoenix_MKDS-1,5-2-5.08_1x02_P5.08mm_Horizontal
- removed J18: Boton 3 sgn, TerminalBlock_Phoenix:TerminalBlock_Phoenix_MKDS-1,5-2-5.08_1x02_P5.08mm_Horizontal
- moved EN1 134.9 mm to (719.3, 177.4)
- moved GND_2 118.1 mm to (717.5, 59.5)
- moved GPIO12 109.2 mm to (717.8, 76.9)
- moved GPIO36 106.2 mm to (719.0, 167.2)
- moved VIN1 104.2 mm to (717.8, 50.7)
- moved GPIO13 101.7 mm to (717.8, 68.1)
- moved GPIO34 100.5 mm to (717.9, 149.5)
- moved GPIO14 99.1 mm to (717.7, 85.3)
- moved GPIO39 98.1 mm to (718.0, 158.7)
- moved GPIO35 93.2 mm to (717.9, 139.3)
- moved GPIO32 90.9 mm to (717.7, 129.0)
- moved GPIO23 90.7 mm to (688.7, 176.6)
- moved GPIO25 90.2 mm to (717.5, 112.5)
- moved GPIO1 89.7 mm to (687.8, 157.1)
- moved GND_1 89.0 mm to (685.4, 56.5)
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Connections:
- C12 pad 1: Net-(J14-Pin_1) -> Net-(GPIO34-Pin_1)
- C14 pad 1: Net-(J16-Pin_1) -> Net-(GPIO14-Pin_1)
- GPIO14 pad 1: unconnected-(GPIO14-Pin_1-Pad1) -> Net-(GPIO14-Pin_1)
- GPIO23 pad 1: unconnected-(GPIO23-Pin_1-Pad1) -> Net-(GPIO23-Pin_1)
- GPIO25 pad 1: unconnected-(GPIO25-Pin_1-Pad1) -> Net-(GPIO25-Pin_1)
- GPIO26 pad 1: unconnected-(GPIO26-Pin_1-Pad1) -> Net-(GPIO14-Pin_1)
- GPIO27 pad 1: unconnected-(GPIO27-Pin_1-Pad1) -> Net-(GPIO14-Pin_1)
- GPIO32 pad 1: unconnected-(GPIO32-Pin_1-Pad1) -> Net-(GPIO32-Pin_1)
- GPIO33 pad 1: unconnected-(GPIO33-Pin_1-Pad1) -> Net-(GPIO33-Pin_1)
- GPIO34 pad 1: unconnected-(GPIO34-Pin_1-Pad1) -> Net-(GPIO34-Pin_1)
- GPIO35 pad 1: unconnected-(GPIO35-Pin_1-Pad1) -> Net-(GPIO34-Pin_1)
- J3 pad 2: Net-(J14-Pin_2) -> Net-(GPIO34-Pin_1)
- J4 pad 2: Net-(J15-Pin_2) -> Net-(GPIO34-Pin_1)
- J5 pad 2: Net-(J16-Pin_2) -> Net-(GPIO14-Pin_1)
- J6 pad 2: Net-(J17-Pin_2) -> Net-(GPIO14-Pin_1)
- J7 pad 2: Net-(J18-Pin_2) -> Net-(GPIO14-Pin_1)
- U1 pad 1: unconnected-(U1-Pad1) -> Net-(GPIO23-Pin_1)
- U10 pad 2: Net-(J16-Pin_1) -> Net-(GPIO14-Pin_1)
- U2 pad 1: unconnected-(U2-Pad1) -> Net-(GPIO32-Pin_1)
- U3 pad 1: unconnected-(U3-Pad1) -> Net-(GPIO33-Pin_1)
- U4 pad 1: unconnected-(U4-Pad1) -> Net-(GPIO25-Pin_1)
- U9 pad 2: Net-(J14-Pin_1) -> Net-(GPIO34-Pin_1)

Commit message: Actualización de PCB
Parts:
- added D8: 1N4001, Diode_THT:D_DO-41_SOD81_P10.16mm_Horizontal, F.Cu at (331.6, 68.5)
- added D9: 1N4001, Diode_THT:D_DO-41_SOD81_P10.16mm_Horizontal, F.Cu at (330.8, 123.1)
- added R11: 1000, Resistor_THT:R_Axial_DIN0207_L6.3mm_D2.5mm_P10.16mm_Horizontal, F.Cu at (398.1, 247.4)
- added R12: 1000, Resistor_THT:R_Axial_DIN0207_L6.3mm_D2.5mm_P10.16mm_Horizontal, F.Cu at (499.2, 240.4)
- added R13: 1000, Resistor_THT:R_Axial_DIN0207_L6.3mm_D2.5mm_P10.16mm_Horizontal, F.Cu at (595.4, 238.4)
- added R14: 1000, Resistor_THT:R_Axial_DIN0207_L6.3mm_D2.5mm_P10.16mm_Horizontal, F.Cu at (716.4, 243.1)
- R10, R4, R6, R8: value 450 -> 500
- R3, R5, R7, R9: value 150 -> 100
- moved R8 28.0 mm to (622.8, 225.1), turned to 180 degrees
- moved U3 22.8 mm to (594.6, 227.9)
- moved C4 22.6 mm to (342.1, 80.2)
- moved R10 17.5 mm to (735.8, 241.6)
- moved U4 17.5 mm to (721.5, 234.0)
- moved U2 16.8 mm to (501.9, 232.5), turned to 180 degrees
- moved C6 16.7 mm to (339.6, 136.1)
- moved U1 8.14 mm to (402.8, 229.7)
- moved K3 2.92 mm to (595.0, 283.0)
- moved R5 2.41 mm to (518.5, 240.3)
Connections:
- C4 pad 1: Net-(U5-VO) -> Net-(D8-K)
- C7 pad 1: Net-(U5-VO) -> Net-(D8-K)
- C9 pad 1: Net-(U5-VO) -> Net-(D8-K)
- K5 pad 9: Net-(U5-VO) -> Net-(D8-K)
- K6 pad 3: Net-(U5-VO) -> unconnected-(K6-Pad3)
- K6 pad 4: unconnected-(K6-Pad4) -> Net-(D8-K)
- U1 pad 3: Net-(Q1-B) -> Net-(R11-Pad2)
- U2 pad 3: Net-(Q2-B) -> Net-(R12-Pad1)
- U3 pad 3: Net-(Q3-B) -> Net-(R13-Pad1)
- U4 pad 3: Net-(Q4-B) -> Net-(R14-Pad1)
- U5 pad 3: Net-(U5-VO) -> Net-(D8-A)
- U6 pad 3: Net-(D3-K) -> Net-(D9-A)
- U7 pad 1: Net-(U5-VO) -> Net-(D8-K)
- U8 pad 1: Net-(U5-VO) -> Net-(D8-K)

Commit message: Organización de elementos
Parts:
- added BT1: Battery, Battery:BatteryHolder_Keystone_1060_1x2032, F.Cu at (288.6, 115.8)
- added C15: 0.1 μF, Capacitor_THT:C_Disc_D3.0mm_W1.6mm_P2.50mm, F.Cu at (53.3, -82.2)
- added C16: 0.22 μF, Capacitor_THT:C_Disc_D3.0mm_W1.6mm_P2.50mm, F.Cu at (36.4, -82.3)
- added D10: 1N4001, Diode_THT:D_DO-41_SOD81_P10.16mm_Horizontal, F.Cu at (44.6, -62.0)
- added D11: 1N4001, Diode_THT:D_DO-41_SOD81_P10.16mm_Horizontal, F.Cu at (44.6, -76.6)
- added D12: 11 V, Diode_THT:D_DO-41_SOD81_P10.16mm_Horizontal, F.Cu at (-150.3, -79.1)
- added D13: 1N4001, Diode_THT:D_DO-41_SOD81_P10.16mm_Horizontal, F.Cu at (-136.1, -78.9)
- added D14: LED, LED_THT:LED_D3.0mm, F.Cu at (-141.6, -101.5)
- added D15: 1N4001, Diode_THT:D_DO-41_SOD81_P10.16mm_Horizontal, F.Cu at (62.9, -92.6)
- added D16: 1N4001, Diode_THT:D_DO-41_SOD81_P10.16mm_Horizontal, F.Cu at (-34.5, -81.6)
- added HS1: Heatsink, Heatsink:Heatsink_125x35x50mm_3xFixationM3, F.Cu at (149.0, 25.8)
- added HS2: Heatsink, Heatsink:Heatsink_125x35x50mm_3xFixationM3, F.Cu at (150.4, 163.5)
- added J14: + de la bateria, TerminalBlock_Phoenix:TerminalBlock_Phoenix_MKDS-1,5-2-5.08_1x02_P5.08mm_Horizontal, F.Cu at (-119.1, -43.4)
- added J15: - de la bateria, TerminalBlock_Phoenix:TerminalBlock_Phoenix_MKDS-1,5-2-5.08_1x02_P5.08mm_Horizontal, F.Cu at (-158.0, -44.0)
- added K7: SANYOU_SRD_Form_C, Relay_THT:Relay_SPDT_SANYOU_SRD_Series_Form_C, F.Cu at (-23.9, -86.8)
- added Q5: BC558, Package_TO_SOT_THT:TO-92_Inline, F.Cu at (-90.4, -78.5)
- added Q6: BC558, Package_TO_SOT_THT:TO-92_Inline, F.Cu at (-68.0, -96.0)
- added Q7: 2N2222A, Package_TO_SOT_THT:TO-92, F.Cu at (-47.8, -111.8)
- added R15: 100 Ω 2W, Resistor_THT:R_Axial_DIN0617_L17.0mm_D6.0mm_P25.40mm_Horizontal, F.Cu at (2.18, -80.4)
- added R16: 100 Ω 2W, Resistor_THT:R_Axial_DIN0617_L17.0mm_D6.0mm_P25.40mm_Horizontal, F.Cu at (78.4, -92.8)
- added R17: 330K, Resistor_THT:R_Axial_DIN0309_L9.0mm_D3.2mm_P12.70mm_Horizontal, F.Cu at (-90.5, -96.0)
- added R18: 4.3K, Resistor_THT:R_Axial_DIN0309_L9.0mm_D3.2mm_P12.70mm_Horizontal, F.Cu at (-97.2, -119.4)
- added R19: 6.8K, Resistor_THT:R_Axial_DIN0309_L9.0mm_D3.2mm_P12.70mm_Horizontal, F.Cu at (-68.9, -112.5)
- added R20: 10K, Resistor_THT:R_Axial_DIN0309_L9.0mm_D3.2mm_P12.70mm_Horizontal, F.Cu at (-114.7, -78.9)
- added R21: 220, Resistor_THT:R_Axial_DIN0309_L9.0mm_D3.2mm_P12.70mm_Horizontal, F.Cu at (-33.6, -74.0)
- added R22: 330K, Resistor_THT:R_Axial_DIN0309_L9.0mm_D3.2mm_P12.70mm_Horizontal, F.Cu at (-123.9, -100.3)
- added REF**: MountingHole_3.2mm_M3, MountingHole:MountingHole_3.2mm_M3, F.Cu at (-54.1, 81.4)
- added REF**: MountingHole_3.2mm_M3, MountingHole:MountingHole_3.2mm_M3, F.Cu at (-52.7, 135.9)
- added REF**: MountingHole_3.2mm_M3, MountingHole:MountingHole_3.2mm_M3, F.Cu at (-52.6, 123.9)
- added REF**: MountingHole_3.2mm_M3, MountingHole:MountingHole_3.2mm_M3, F.Cu at (-54.7, 69.7)
- added U11: LM7812_TO220, Package_TO_SOT_THT:TO-220-3_Vertical, F.Cu at (42.1, -92.1)
- added U12: DS1307+, Package_DIP:DIP-8_W7.62mm, F.Cu at (279.6, 141.8)
- added Y1: Crystal, Crystal:Crystal_C26-LF_D2.1mm_L6.5mm_Horizontal, F.Cu at (301.0, 144.8)
- U10, U9: footprint Package_TO_SOT_THT:TO-220-3_Horizontal_TabDown -> Package_TO_SOT_THT:TO-220-3_Vertical
- moved J2 405.0 mm to (-53.8, 245.4)
- moved D7 373.5 mm to (-56.8, 208.2), turned to -90 degrees
- moved J6 363.0 mm to (303.8, 245.4)
- moved J5 359.1 mm to (265.2, 244.9)
- moved J7 359.1 mm to (339.6, 245.4)
- moved C14 329.9 mm to (166.6, 18.9), turned to 90 degrees
- moved C12 327.5 mm to (166.3, -14.9), turned to -90 degrees
- moved J3 317.3 mm to (197.7, 243.2)
- moved J4 315.2 mm to (229.8, 244.4)
- moved U10 313.3 mm to (155.6, 16.5), turned to 90 degrees
- moved U9 307.2 mm to (155.7, -7.20), turned to 90 degrees
- moved C13 289.9 mm to (166.7, 9.73), turned to -90 degrees
- moved C11 278.3 mm to (166.3, -5.95), turned to 90 degrees
- moved K6 246.6 mm to (-106.3, 116.5), turned to -90 degrees
- moved C10 246.3 mm to (166.6, 57.5), turned to -90 degrees
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Connections:
- GND_2 pad 1: unconnected-(GND_2-Pin_1-Pad1) -> Net-(BT1--)
- GPIO21 pad 1: unconnected-(GPIO21-Pin_1-Pad1) -> Net-(GPIO21-Pin_1)
- GPIO22 pad 1: unconnected-(GPIO22-Pin_1-Pad1) -> Net-(GPIO22-Pin_1)
Other:
- board outline added: 836.7 x 424.2 mm
- board text added: "120 VAC"
- board text added: "Bateria 12 VDC"
- board text added: "Boton 1"
- board text added: "Boton 2"
- board text added: "Boton 3"
- board text added: "Salida 1"
- board text added: "Salida 2"
- board text added: "Salida 3"
- board text added: "Salida 4"
- board text added: "Sensor IN"
- board text added: "Sensor OUT"
