File: Panel_PCB/Panel_PCB.kicad_pcb (KiCad board)
At the start: 2 copper layers, 836.7 x 424.2 mm, 135 parts, among them J1 AC, J10 Relay 3, J11 Relay 4, J12 AC, J13 AC, J14 + de la bateria, J15 - de la bateria, J2 Bateria, J3 Sensor IN, J4 Sensor OUT, J5 Boton 1, J6 Boton 2, J7 Boton 3, J8 Relay 1, J9 Relay 2, K1 SANYOU_SRD_Form_C, K2 SANYOU_SRD_Form_C, K3 SANYOU_SRD_Form_C, K4 SANYOU_SRD_Form_C, K5 EC2-4.5SNU, K6 SANYOU_SRD_Form_C, K7 SANYOU_SRD_Form_C, Q1 2N2222A, Q2 2N2222A, Q3 2N2222A, Q4 2N2222A, Q5 BC558, Q6 BC558, Q7 2N2222A, U1 TLP291, U10 LM1117T-3.3, U11 LM7812_TO220, U12 DS1307+, U2 TLP291, U3 TLP291, U4 TLP291, U5 LM7812_TO220, U6 LM7812_TO220, U7 LM7805_TO220, U8 LM7805_TO220, U9 LM1117T-3.3, Y1 Crystal

Commit message: Comparador de voltaje (para el cargador de batería)
Parts:
- removed D12: 11 V, Diode_THT:D_DO-41_SOD81_P10.16mm_Horizontal
- removed D13: 1N4001, Diode_THT:D_DO-41_SOD81_P10.16mm_Horizontal
- removed D14: LED, LED_THT:LED_D3.0mm
- removed J14: + de la bateria, TerminalBlock_Phoenix:TerminalBlock_Phoenix_MKDS-1,5-2-5.08_1x02_P5.08mm_Horizontal
- removed J15: - de la bateria, TerminalBlock_Phoenix:TerminalBlock_Phoenix_MKDS-1,5-2-5.08_1x02_P5.08mm_Horizontal
- removed Q5, Q6: BC558, Package_TO_SOT_THT:TO-92_Inline
- removed R20: 10K, Resistor_THT:R_Axial_DIN0309_L9.0mm_D3.2mm_P12.70mm_Horizontal
- removed R22: 330K, Resistor_THT:R_Axial_DIN0309_L9.0mm_D3.2mm_P12.70mm_Horizontal
- added U13: LM311, Package_DIP:DIP-8_W7.62mm, F.Cu at (-53.0, -81.2)
- R17: value 330K -> 1K
- R18: value 4.3K -> 2K
- moved D15 131.7 mm to (-68.6, -85.7), turned to 0 degrees
- moved R16 131.2 mm to (-52.7, -87.0)
- moved D10 117.7 mm to (-68.6, -94.2), turned to 0 degrees
- moved D11 114.0 mm to (-68.6, -89.9), turned to 0 degrees
- moved C15 95.6 mm to (-42.3, -81.7), turned to 0 degrees
- moved C16 78.8 mm to (-42.3, -78.5), turned to 0 degrees
- moved U11 78.1 mm to (-35.0, -79.3)
- moved R15 56.6 mm to (-52.7, -94.6)
- moved R21 43.1 mm to (-68.9, -98.7), turned to 0 degrees
- moved K7 34.9 mm to (-52.6, -106.8)
- moved D16 34.1 mm to (-68.6, -81.4), turned to 0 degrees
- moved R18 30.4 mm to (-68.9, -108.2), turned to 0 degrees
- moved R17 27.4 mm to (-68.9, -112.9)
- moved Q7 16.3 mm to (-31.5, -112.0)
- moved R19 9.13 mm to (-68.9, -103.4)
Connections:
- C15 pad 2: Net-(D10-K) -> Net-(D1--)
- C16 pad 2: Net-(D10-K) -> Net-(D1--)
- D10 pad 1: Net-(D10-K) -> Net-(D1--)
- GPIO18 pad 1: unconnected-(GPIO18-Pin_1-Pad1) -> Net-(GPIO18-Pin_1)
- GPIO39 pad 1: unconnected-(GPIO39-Pin_1-Pad1) -> Net-(GPIO39-Pin_1)
- K7 pad 2: Net-(D16-K) -> Net-(D16-A)
- K7 pad 5: Net-(D16-A) -> Net-(D16-K)
- Q7 pad 1: Net-(D12-A) -> Net-(Q7-E)
- R16 pad 2: unconnected-(R16-Pad2) -> Net-(D7-A)
- R17 pad 1: Net-(Q6-B) -> Net-(D16-K)
- R17 pad 2: Net-(Q5-C) -> Net-(C1-Pad1)
- R18 pad 1: Net-(D12-A) -> Net-(GPIO34-Pin_1)
- R18 pad 2: Net-(Q5-C) -> Net-(GPIO39-Pin_1)
- R19 pad 2: Net-(Q6-C) -> Net-(GPIO18-Pin_1)
- R21 pad 1: Net-(D16-K) -> Net-(Q7-E)
- R21 pad 2: Net-(J14-Pin_1) -> Net-(D1--)

Commit message: Nuevo esquematico (falta boost converter de 12V a 13.5V
Parts:
- removed C1: 35V 4700μF, Capacitor_THT:C_Radial_D18.0mm_H35.5mm_P7.50mm
- removed C3, C5: 0.22 μF, Capacitor_THT:C_Disc_D3.0mm_W1.6mm_P2.50mm
- removed C4, C6: 0.1 μF, Capacitor_THT:C_Disc_D3.0mm_W1.6mm_P2.50mm
- removed F2: Fuse_Small, Fuse:Fuseholder_Cylinder-5x20mm_Schurter_0031_8201_Horizontal_Open
- removed HS2: Heatsink, Heatsink:Heatsink_125x35x50mm_3xFixationM3
- removed J12, J13: AC, TerminalBlock_Phoenix:TerminalBlock_Phoenix_MKDS-1,5-2-5.08_1x02_P5.08mm_Horizontal
- removed K6: SANYOU_SRD_Form_C, Relay_THT:Relay_SPDT_SANYOU_SRD_Series_Form_C
- removed R1: 100 Ω 2W, Resistor_THT:R_Axial_DIN0617_L17.0mm_D6.0mm_P25.40mm_Horizontal
- removed REF** (x4): MountingHole_3.2mm_M3, MountingHole:MountingHole_3.2mm_M3
- removed U5, U6: LM7812_TO220, Package_TO_SOT_THT:TO-220-3_Vertical
- D1: value KBP204G -> 1N4001; footprint Diode_THT:Diode_Bridge_Vishay_KBPM -> Diode_THT:D_DO-41_SOD81_P10.16mm_Horizontal
- J1: value AC -> DC
- moved R18 286.1 mm to (211.1, -49.2), turned to 90 degrees
- moved D9 250.0 mm to (170.4, -66.3), turned to 180 degrees
- moved D8 242.5 mm to (136.5, -104.3), turned to 0 degrees
- moved U13 241.0 mm to (187.6, -68.2)
- moved D1 225.0 mm to (136.5, -108.5), turned to 0 degrees
- moved R16 129.1 mm to (72.6, -55.8)
- moved D10 116.2 mm to (43.5, -63.4), turned to 180 degrees
- moved R21 110.6 mm to (-33.9, 6.26)
- moved D11 108.0 mm to (33.6, -55.2)
- moved Q7 105.1 mm to (-29.4, -6.98)
- moved R19 97.1 mm to (-54.4, -7.37)
- moved C16 92.0 mm to (49.4, -70.7), turned to 90 degrees
- moved C15 91.5 mm to (49.2, -79.9), turned to -90 degrees
- moved K7 77.6 mm to (-29.4, -32.7)
- moved U11 66.1 mm to (30.7, -72.3), turned to 90 degrees
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Connections:
- C10 pad 2: Net-(D1--) -> Net-(D10-K)
- C11 pad 2: Net-(D1--) -> Net-(D10-K)
- C12 pad 2: Net-(D1--) -> Net-(D10-K)
- C13 pad 2: Net-(D1--) -> Net-(D10-K)
- C14 pad 2: Net-(D1--) -> Net-(D10-K)
- C15 pad 2: Net-(D1--) -> Net-(D10-K)
- C16 pad 2: Net-(D1--) -> Net-(D10-K)
- C2 pad 2: Net-(D1--) -> Net-(D10-K)
- C7 pad 1: Net-(D8-K) -> Net-(D2-K)
- C7 pad 2: Net-(D1--) -> Net-(D10-K)
- C8 pad 2: Net-(D1--) -> Net-(D10-K)
- C9 pad 1: Net-(D8-K) -> Net-(D2-K)
- C9 pad 2: Net-(D1--) -> Net-(D10-K)
- D1 pad 1: Net-(D1-+) -> Net-(D1-K)
- D1 pad 2: Net-(D1-Pad2) -> Net-(D1-A)
- D10 pad 1: Net-(D1--) -> Net-(D10-K)
- D2 pad 2: Net-(D1--) -> Net-(D10-K)
- D3 pad 1: Net-(D3-K) -> Net-(D2-K)
- D4 pad 1: Net-(D3-K) -> Net-(D2-K)
- D5 pad 1: Net-(D3-K) -> Net-(D2-K)
- D6 pad 1: Net-(D3-K) -> Net-(D2-K)
- D8 pad 2: Net-(D8-A) -> Net-(D10-K)
- D9 pad 1: Net-(D3-K) -> Net-(D9-K)
- D9 pad 2: Net-(D9-A) -> Net-(D1-K)
- F1 pad 2: Net-(J12-Pin_1) -> Net-(D1-A)
- GND_1 pad 1: Net-(D1--) -> Net-(D10-K)
- J1 pad 1: Net-(J1-Pin_1) -> Net-(D8-K)
- J2 pad 2: Net-(D1--) -> Net-(D10-K)
- J3 pad 1: Net-(D1--) -> Net-(D10-K)
- J4 pad 1: Net-(D1--) -> Net-(D10-K)
- J5 pad 1: Net-(D1--) -> Net-(D10-K)
- J6 pad 1: Net-(D1--) -> Net-(D10-K)
- J7 pad 1: Net-(D1--) -> Net-(D10-K)
- K1 pad 5: Net-(D3-K) -> Net-(D2-K)
- K2 pad 5: Net-(D3-K) -> Net-(D2-K)
- K3 pad 5: Net-(D3-K) -> Net-(D2-K)
- K4 pad 5: Net-(D3-K) -> Net-(D2-K)
- K5 pad 1: Net-(J12-Pin_1) -> Net-(D1-K)
- K5 pad 12: Net-(J1-Pin_1) -> Net-(D10-K)
- K5 pad 4: Net-(C1-Pad1) -> Net-(D1-K)
- K5 pad 9: Net-(D8-K) -> Net-(K5-Pad5)
- K7 pad 1: Net-(K5-Pad5) -> unconnected-(K7-Pad1)
- R10 pad 1: Net-(D3-K) -> Net-(D2-K)
- R17 pad 2: Net-(C1-Pad1) -> Net-(D1-K)
- R21 pad 2: Net-(D1--) -> Net-(D10-K)
- R3 pad 2: Net-(D1--) -> Net-(D10-K)
- R4 pad 1: Net-(D3-K) -> Net-(D2-K)
- R5 pad 2: Net-(D1--) -> Net-(D10-K)
- R6 pad 1: Net-(D3-K) -> Net-(D2-K)
- R7 pad 2: Net-(D1--) -> Net-(D10-K)
- R8 pad 1: Net-(D3-K) -> Net-(D2-K)
- R9 pad 2: Net-(D1--) -> Net-(D10-K)
- U1 pad 2: Net-(D1--) -> Net-(D10-K)
- U10 pad 1: Net-(D1--) -> Net-(D10-K)
- U13 pad 1: Net-(D1--) -> Net-(D10-K)
- U13 pad 2: Net-(D8-K) -> Net-(D9-K)
- U13 pad 4: unconnected-(U13-V--Pad4) -> Net-(D10-K)
- U13 pad 8: unconnected-(U13-V+-Pad8) -> Net-(D2-K)
- U2 pad 2: Net-(D1--) -> Net-(D10-K)
- U3 pad 2: Net-(D1--) -> Net-(D10-K)
- U4 pad 2: Net-(D1--) -> Net-(D10-K)
- U7 pad 1: Net-(D8-K) -> Net-(D2-K)
- U7 pad 2: Net-(D1--) -> Net-(D10-K)
- U8 pad 1: Net-(D8-K) -> Net-(D2-K)
- U8 pad 2: Net-(D1--) -> Net-(D10-K)
- U9 pad 1: Net-(D1--) -> Net-(D10-K)

Commit message: Ajustes al esquemático
Parts:
- added R1: 330, Resistor_THT:R_Axial_DIN0207_L6.3mm_D2.5mm_P10.16mm_Horizontal, F.Cu at (410.4, 147.7)
- added R20: 330, Resistor_THT:R_Axial_DIN0207_L6.3mm_D2.5mm_P10.16mm_Horizontal, F.Cu at (477.5, 141.0)
- added R22: 330, Resistor_THT:R_Axial_DIN0207_L6.3mm_D2.5mm_P10.16mm_Horizontal, F.Cu at (528.2, 140.3)
- added R23: 330, Resistor_THT:R_Axial_DIN0207_L6.3mm_D2.5mm_P10.16mm_Horizontal, F.Cu at (598.7, 143.7)
- R19: value 6.8K -> 330
- R3, R5, R7, R9: value 100 -> 1000
Connections:
- U1 pad 1: Net-(GPIO23-Pin_1) -> Net-(R1-Pad2)
- U2 pad 1: Net-(GPIO32-Pin_1) -> Net-(R20-Pad2)
- U3 pad 1: Net-(GPIO33-Pin_1) -> Net-(R22-Pad2)
- U4 pad 1: Net-(GPIO25-Pin_1) -> Net-(R23-Pad2)

Commit message: Actualización de placa
Parts:
- removed 3V3, EN1, GND_1, GND_2, GPIO1, GPIO12, GPIO13, GPIO14, GPIO15, GPIO16, GPIO17, GPIO18, GPIO19, GPIO2, GPIO21, GPIO22, GPIO23, GPIO25, GPIO26, GPIO27, GPIO3, GPIO32, GPIO33, GPIO34, GPIO35, GPIO36, GPIO39, GPIO4, GPIO5, VIN1: ~, Connector_Wire:SolderWire-0.75sqmm_1x01_D1.25mm_OD2.3mm
- added J12: Terminal A, TerminalBlock:TerminalBlock_Xinya_XY308-2.54-15P_1x15_P2.54mm_Horizontal, F.Cu at (419.6, 47.0)
- added J13: Terminal B, TerminalBlock:TerminalBlock_Xinya_XY308-2.54-15P_1x15_P2.54mm_Horizontal, F.Cu at (445.0, 82.5)
Other:
- board text added: "3V3 GND_1 GPIO15 GPIO2 GPIO4 GPIO16 GPIO17 GPIO5 GPIO18 GPIO19 GPIO21 GPIO3 GPIO1 GPIO22 GPIO23"
- board text added: "VIN1 GND_2 GPIO13 GPIO12 GPIO14 GPIO27 GPIO26 GPIO25 GPIO33 GPIO32 GPIO35 GPIO34 GPIO39 GPIO36 EN1"

Commit message: Información para usar el control remoto
Parts:
- added C1: 100 μF, Capacitor_THT:C_Disc_D3.0mm_W1.6mm_P2.50mm, F.Cu at (437.3, -49.8)
- added C3: 10 μF, Capacitor_THT:C_Disc_D3.0mm_W1.6mm_P2.50mm, F.Cu at (437.3, -46.7)
- added C4: 25V 4700μF, Capacitor_THT:C_Radial_D18.0mm_H35.5mm_P7.50mm, F.Cu at (410.0, -91.5)
- added C5: 25V 4700μF, Capacitor_THT:C_Radial_D18.0mm_H35.5mm_P7.50mm, F.Cu at (410.0, -71.9)
- added C6: 25V 4700μF, Capacitor_THT:C_Radial_D18.0mm_H35.5mm_P7.50mm, F.Cu at (410.0, -52.4)
- added D12: 1N4001, Diode_THT:D_DO-41_SOD81_P10.16mm_Horizontal, F.Cu at (425.4, -99.1)
- added D13: 1N4001, Diode_THT:D_DO-41_SOD81_P10.16mm_Horizontal, F.Cu at (425.4, -94.9)
- added D14: 1N4001, Diode_THT:D_DO-41_SOD81_P10.16mm_Horizontal, F.Cu at (425.4, -90.6)
- added D19: 1N4001, Diode_THT:D_DO-41_SOD81_P10.16mm_Horizontal, F.Cu at (425.4, -86.4)
- added J14: Boton D (4), TerminalBlock_Phoenix:TerminalBlock_Phoenix_MKDS-1,5-2-5.08_1x02_P5.08mm_Horizontal, F.Cu at (427.1, -57.1)
- added J15: Control remoto, TerminalBlock:TerminalBlock_Xinya_XY308-2.54-7P_1x07_P2.54mm_Horizontal, F.Cu at (505.8, -57.7)
- added R15: 10KΩ, Resistor_THT:R_Axial_DIN0207_L6.3mm_D2.5mm_P10.16mm_Horizontal, F.Cu at (425.1, -78.2)
- added R2: 10KΩ, Resistor_THT:R_Axial_DIN0207_L6.3mm_D2.5mm_P10.16mm_Horizontal, F.Cu at (425.1, -82.2)
- added R24: 10K, Resistor_THT:R_Axial_DIN0207_L6.3mm_D2.5mm_P10.16mm_Horizontal, F.Cu at (425.1, -74.1)
- added R25: 10K, Resistor_THT:R_Axial_DIN0207_L6.3mm_D2.5mm_P10.16mm_Horizontal, F.Cu at (425.1, -70.1)
- added R26: 10K, Resistor_THT:R_Axial_DIN0309_L9.0mm_D3.2mm_P12.70mm_Horizontal, F.Cu at (425.1, -65.7)
- added U5: LM7805_TO220, Package_TO_SOT_THT:TO-220-3_Vertical, F.Cu at (439.0, -59.4)
- added U6: LM1117T-3.3, Package_TO_SOT_THT:TO-220-3_Vertical, F.Cu at (439.0, -53.4)
- C2: value 35V 4700μF -> 25V 4700μF
- J5: value Boton 1 -> Boton A (1)
- J6: value Boton 2 -> Boton B (2)
- J7: value Boton 3 -> Boton C (3)
- R10, R4, R6, R8: value 500 -> 1000
- R18: value 2K -> 10K
- R21: value 220 -> 50
- R3, R5, R7, R9: value 1000 -> 50; footprint Resistor_THT:R_Axial_DIN0207_L6.3mm_D2.5mm_P10.16mm_Horizontal -> Resistor_THT:R_Axial_DIN0309_L9.0mm_D3.2mm_P12.70mm_Horizontal
Connections:
- C10 pad 1: Net-(J13-Pin_15) -> Net-(J12-Pin_11)
- C10 pad 2: Net-(D10-K) -> Net-(D19-A)
- C11 pad 2: Net-(D10-K) -> Net-(D19-A)
- C12 pad 1: Net-(J13-Pin_4) -> Net-(J3-Pin_1)
- C12 pad 2: Net-(D10-K) -> Net-(D19-A)
- C13 pad 2: Net-(D10-K) -> Net-(D19-A)
- C14 pad 1: Net-(J13-Pin_10) -> Net-(J14-Pin_1)
- C14 pad 2: Net-(D10-K) -> Net-(D19-A)
- C2 pad 1: Net-(D2-K) -> Net-(D12-A)
- C2 pad 2: Net-(D10-K) -> Net-(D19-A)
- C7 pad 1: Net-(D2-K) -> Net-(D12-A)
- C7 pad 2: Net-(D10-K) -> Net-(D19-A)
- C8 pad 2: Net-(D10-K) -> Net-(D19-A)
- C9 pad 1: Net-(D2-K) -> Net-(D12-A)
- C9 pad 2: Net-(D10-K) -> Net-(D19-A)
- D16 pad 1: Net-(D16-K) -> Net-(D1-K)
- D3 pad 1: Net-(D2-K) -> Net-(D12-A)
- D4 pad 1: Net-(D2-K) -> Net-(D12-A)
- D5 pad 1: Net-(D2-K) -> Net-(D12-A)
- D6 pad 1: Net-(D2-K) -> Net-(D12-A)
- D7 pad 1: Net-(D7-K) -> Net-(D12-A)
- J1 pad 1: Net-(D8-K) -> Net-(D19-A)
- J12 pad 14: Net-(J12-Pin_14) -> Net-(J12-Pin_11)
- J12 pad 2: Net-(D10-K) -> Net-(D19-A)
- J13 pad 11: Net-(J13-Pin_10) -> Net-(J13-Pin_11)
- J13 pad 13: unconnected-(J13-Pin_13-Pad13) -> Net-(J13-Pin_13)
- J13 pad 15: Net-(J13-Pin_15) -> Net-(J12-Pin_11)
- J13 pad 5: Net-(J13-Pin_4) -> Net-(J13-Pin_5)
- J13 pad 9: Net-(J13-Pin_10) -> Net-(J13-Pin_9)
- J2 pad 1: Net-(D7-A) -> Net-(J2-Pin_1)
- J2 pad 2: Net-(D10-K) -> Net-(D19-A)
- J3 pad 1: Net-(D10-K) -> Net-(J3-Pin_1)
- J4 pad 1: Net-(D10-K) -> Net-(J3-Pin_1)
- J4 pad 2: Net-(J13-Pin_4) -> Net-(J13-Pin_5)
- J5 pad 1: Net-(D10-K) -> Net-(J14-Pin_1)
- J5 pad 2: Net-(J13-Pin_10) -> Net-(J13-Pin_9)
- J6 pad 1: Net-(D10-K) -> Net-(J14-Pin_1)
- J7 pad 1: Net-(D10-K) -> Net-(J14-Pin_1)
- J7 pad 2: Net-(J13-Pin_10) -> Net-(J13-Pin_11)
- K1 pad 5: Net-(D2-K) -> Net-(D12-A)
- K2 pad 5: Net-(D2-K) -> Net-(D12-A)
- K3 pad 5: Net-(D2-K) -> Net-(D12-A)
- K4 pad 5: Net-(D2-K) -> Net-(D12-A)
- K5 pad 10: Net-(D7-K) -> Net-(J2-Pin_1)
- K5 pad 12: Net-(D10-K) -> Net-(D19-A)
- K5 pad 5: Net-(K5-Pad5) -> Net-(D12-A)
- K5 pad 9: Net-(K5-Pad5) -> Net-(D7-A)
- K7 pad 1: unconnected-(K7-Pad1) -> Net-(D1-A)
- K7 pad 3: Net-(K7-Pad3) -> Net-(J2-Pin_1)
- K7 pad 5: Net-(D16-K) -> Net-(D1-K)
- R10 pad 1: Net-(D2-K) -> Net-(D12-A)
- R18 pad 1: Net-(J13-Pin_4) -> Net-(D12-K)
- R18 pad 2: Net-(J13-Pin_3) -> Net-(R18-Pad2)
- R21 pad 2: Net-(D10-K) -> Net-(U13-V-)
- R3 pad 2: Net-(D10-K) -> Net-(D19-A)
- R4 pad 1: Net-(D2-K) -> Net-(D12-A)
- R5 pad 2: Net-(D10-K) -> Net-(D19-A)
- R6 pad 1: Net-(D2-K) -> Net-(D12-A)
- R7 pad 2: Net-(D10-K) -> Net-(D19-A)
- R8 pad 1: Net-(D2-K) -> Net-(D12-A)
- R9 pad 2: Net-(D10-K) -> Net-(D19-A)
- U1 pad 2: Net-(D10-K) -> Net-(D19-A)
- U10 pad 1: Net-(D10-K) -> Net-(D19-A)
- U10 pad 2: Net-(J13-Pin_10) -> Net-(J14-Pin_1)
- U12 pad 5: Net-(J12-Pin_11) -> Net-(U12-SDA)
- U12 pad 6: Net-(J12-Pin_14) -> Net-(U12-SCL)
- U12 pad 8: Net-(J13-Pin_15) -> Net-(J12-Pin_11)
- U13 pad 1: Net-(D10-K) -> Net-(U13-GND)
- U13 pad 2: Net-(D9-K) -> Net-(J2-Pin_1)
- U13 pad 3: Net-(D7-A) -> Net-(D13-K)
- U13 pad 4: Net-(D10-K) -> Net-(U13-V-)
- U13 pad 7: Net-(J13-Pin_3) -> Net-(R18-Pad2)
- U13 pad 8: Net-(D2-K) -> Net-(D12-K)
- U2 pad 2: Net-(D10-K) -> Net-(D19-A)
- U3 pad 2: Net-(D10-K) -> Net-(D19-A)
- U4 pad 2: Net-(D10-K) -> Net-(D19-A)
- U7 pad 1: Net-(D2-K) -> Net-(D12-A)
- U7 pad 2: Net-(D10-K) -> Net-(D19-A)
- U8 pad 1: Net-(D2-K) -> Net-(D12-A)
- U8 pad 2: Net-(D10-K) -> Net-(D19-A)
- U8 pad 3: Net-(J13-Pin_15) -> Net-(J12-Pin_11)
- U9 pad 1: Net-(D10-K) -> Net-(D19-A)
- U9 pad 2: Net-(J13-Pin_4) -> Net-(J3-Pin_1)
- Y1 pad 1: Net-(U12-X2) -> Net-(U12-X1)
- Y1 pad 2: Net-(U12-X1) -> Net-(U12-X2)

Commit message: Actualización de esquematico
Parts:
- removed HS1: Heatsink, Heatsink:Heatsink_125x35x50mm_3xFixationM3
- added D10: 1N47xxA, Diode_THT:D_DO-41_SOD81_P10.16mm_Horizontal, F.Cu at (585.7, -37.6)
- added D2: 1N47xxA, Diode_THT:D_DO-41_SOD81_P10.16mm_Horizontal, F.Cu at (585.7, -50.4)
- added D8: 1N47xxA, Diode_THT:D_DO-41_SOD81_P10.16mm_Horizontal, F.Cu at (585.7, -46.1)
- added D9: 1N47xxA, Diode_THT:D_DO-41_SOD81_P10.16mm_Horizontal, F.Cu at (585.7, -41.9)
- added R16: 500, Resistor_THT:R_Axial_DIN0207_L6.3mm_D2.5mm_P10.16mm_Horizontal, F.Cu at (599.3, -50.5)
- added R17: 500, Resistor_THT:R_Axial_DIN0207_L6.3mm_D2.5mm_P10.16mm_Horizontal, F.Cu at (599.3, -46.4)
- added R27: 500, Resistor_THT:R_Axial_DIN0207_L6.3mm_D2.5mm_P10.16mm_Horizontal, F.Cu at (599.3, -42.4)
- added R28: 500, Resistor_THT:R_Axial_DIN0207_L6.3mm_D2.5mm_P10.16mm_Horizontal, F.Cu at (599.3, -38.3)
Connections:
- C1 pad 2: Net-(U13-V-) -> Net-(D10-A)
- C11 pad 1: Net-(U10-VI) -> Net-(J15-Pin_2)
- C13 pad 1: Net-(U10-VI) -> Net-(J15-Pin_2)
- C3 pad 2: Net-(U13-V-) -> Net-(D10-A)
- C8 pad 1: Net-(U10-VI) -> Net-(J15-Pin_2)
- J13 pad 10: Net-(J13-Pin_10) -> Net-(D2-K)
- J13 pad 11: Net-(J13-Pin_11) -> Net-(D10-K)
- J13 pad 13: Net-(J13-Pin_13) -> Net-(D8-K)
- J13 pad 9: Net-(J13-Pin_9) -> Net-(D9-K)
- J14 pad 2: Net-(J13-Pin_13) -> Net-(D8-K)
- J15 pad 1: unconnected-(J15-Pin_1-Pad1) -> Net-(D10-A)
- J15 pad 2: unconnected-(J15-Pin_2-Pad2) -> Net-(J15-Pin_2)
- J15 pad 3: unconnected-(J15-Pin_3-Pad3) -> Net-(J15-Pin_3)
- J15 pad 4: unconnected-(J15-Pin_4-Pad4) -> Net-(J15-Pin_4)
- J15 pad 5: unconnected-(J15-Pin_5-Pad5) -> Net-(J15-Pin_5)
- J15 pad 6: unconnected-(J15-Pin_6-Pad6) -> Net-(J15-Pin_6)
- J5 pad 2: Net-(J13-Pin_9) -> Net-(D9-K)
- J6 pad 2: Net-(J13-Pin_10) -> Net-(D2-K)
- J7 pad 2: Net-(J13-Pin_11) -> Net-(D10-K)
- R15 pad 1: Net-(J13-Pin_5) -> Net-(BT1--)
- R15 pad 2: Net-(BT1--) -> Net-(J13-Pin_5)
- R2 pad 1: Net-(J13-Pin_4) -> Net-(BT1--)
- R2 pad 2: Net-(BT1--) -> Net-(J13-Pin_4)
- R21 pad 2: Net-(U13-V-) -> Net-(D10-A)
- R26 pad 2: Net-(U13-V-) -> Net-(D10-A)
- U10 pad 3: Net-(U10-VI) -> Net-(J15-Pin_2)
- U13 pad 4: Net-(U13-V-) -> Net-(D10-A)
- U5 pad 2: Net-(U13-V-) -> Net-(D10-A)
- U6 pad 1: Net-(U13-V-) -> Net-(D10-A)
- U7 pad 3: Net-(U10-VI) -> Net-(J15-Pin_2)
- U9 pad 3: Net-(U10-VI) -> Net-(J15-Pin_2)
