File: Panel_PCB/Panel_PCB.kicad_pcb (KiCad board)
At the start: 2 copper layers, 836.7 x 424.2 mm, 111 parts, among them J1 DC, J10 Relay 3, J11 Relay 4, J12 Terminal A, J13 Terminal B, J14 Boton D (4), J15 Control remoto, J2 Bateria, J3 Sensor IN, J4 Sensor OUT, J5 Boton A (1), J6 Boton B (2), J7 Boton C (3), J8 Relay 1, J9 Relay 2, K1 SANYOU_SRD_Form_C, K2 SANYOU_SRD_Form_C, K3 SANYOU_SRD_Form_C, K4 SANYOU_SRD_Form_C, K5 EC2-4.5SNU, K7 SANYOU_SRD_Form_C, Q1 2N2222A, Q2 2N2222A, Q3 2N2222A, Q4 2N2222A, Q7 2N2222A, U1 TLP291, U10 LM1117T-3.3, U11 LM7812_TO220, U12 DS1307+, U13 LM311, U2 TLP291, U3 TLP291, U4 TLP291, U5 LM7805_TO220, U6 LM1117T-3.3, U7 LM7805_TO220, U8 LM7805_TO220, U9 LM1117T-3.3, Y1 Crystal

Commit message: Corrección de footprint
Parts:
- added R29: 10, Resistor_THT:R_Axial_Power_L60.0mm_W14.0mm_P66.04mm, F.Cu at (224.2, -116.9)
- K5: value EC2-4.5SNU -> G6K-2P-Y
- K6: renamed from K7; value SANYOU_SRD_Form_C -> G5LE-1-E; footprint Relay_THT:Relay_SPDT_SANYOU_SRD_Series_Form_C -> Relay_THT:Relay_SPDT_Omron-G5LE-1
Connections:
- K6 pad 3: Net-(J2-Pin_1) -> Net-(K6-Pad3)

Commit message: Actualizacion de PCB
Parts:
- removed C15: 0.1 μF, Capacitor_THT:C_Disc_D3.0mm_W1.6mm_P2.50mm
- removed C16: 0.22 μF, Capacitor_THT:C_Disc_D3.0mm_W1.6mm_P2.50mm
- removed the D10 at (585.7, -37.6)
- removed the D10 at (43.5, -63.4)
- removed D11, D15: 1N4001, Diode_THT:D_DO-41_SOD81_P10.16mm_Horizontal
- removed the D2 at (66.7, 104.3)
- removed the D2 at (585.7, -50.4)
- removed the D4 at (491.3, 219.3)
- removed the D8 at (136.5, -104.3)
- removed the D8 at (585.7, -46.1)
- removed the D9 at (170.4, -66.3)
- removed the D9 at (585.7, -41.9)
- removed the J9 at (471.0, 245.7)
- removed the R15 at (-6.18, -65.0)
- removed the R15 at (425.1, -78.2)
- removed the R16 at (599.3, -50.5)
- removed the R16 at (72.6, -55.8)
- removed the R17 at (-48.1, -50.7)
- removed the R17 at (599.3, -46.4)
- removed the R2 at (425.1, -82.2)
- removed the R2 at (69.6, 88.9)
- removed the R6 at (456.5, 219.5)
- removed the R7 at (518.4, 220.0)
- removed U11: LM7812_TO220, Package_TO_SOT_THT:TO-220-3_Vertical
- added D10: 1N47xxA, Diode_THT:D_DO-41_SOD81_P10.16mm_Horizontal, F.Cu at (190.3, -94.5)
- added D2: 1N47xxA, Diode_THT:D_DO-41_SOD81_P10.16mm_Horizontal, F.Cu at (190.3, -107.2)
- added D4: 1N4001, Diode_THT:D_DO-41_SOD81_P10.16mm_Horizontal, F.Cu at (249.2, 142.3)
- added D4: 1N4001, Diode_THT:D_DO-41_SOD81_P10.16mm_Horizontal, F.Cu at (178.0, 132.9)
- added D8: 1N47xxA, Diode_THT:D_DO-41_SOD81_P10.16mm_Horizontal, F.Cu at (190.3, -103.0)
- added D9: 1N47xxA, Diode_THT:D_DO-41_SOD81_P10.16mm_Horizontal, F.Cu at (190.3, -98.7)
- added J9: Relay 2, TerminalBlock_Phoenix:TerminalBlock_Phoenix_MKDS-1,5-2-5.08_1x02_P5.08mm_Horizontal, F.Cu at (190.4, 201.8)
- added J9: Relay 2, TerminalBlock_Phoenix:TerminalBlock_Phoenix_MKDS-1,5-2-5.08_1x02_P5.08mm_Horizontal, F.Cu at (248.4, 173.3)
- added R15: 10KΩ, Resistor_THT:R_Axial_DIN0207_L6.3mm_D2.5mm_P10.16mm_Horizontal, F.Cu at (92.8, 54.0)
- added R16: 500, Resistor_THT:R_Axial_DIN0207_L6.3mm_D2.5mm_P10.16mm_Horizontal, F.Cu at (190.1, -68.8)
- added R17: 500, Resistor_THT:R_Axial_DIN0207_L6.3mm_D2.5mm_P10.16mm_Horizontal, F.Cu at (190.1, -64.7)
- added R2: 10KΩ, Resistor_THT:R_Axial_DIN0207_L6.3mm_D2.5mm_P10.16mm_Horizontal, F.Cu at (100.4, 60.8)
- added R6: 1000, Resistor_THT:R_Axial_DIN0207_L6.3mm_D2.5mm_P10.16mm_Horizontal, F.Cu at (177.7, 137.1)
- added R6: 1000, Resistor_THT:R_Axial_DIN0207_L6.3mm_D2.5mm_P10.16mm_Horizontal, F.Cu at (233.1, 165.1)
- added R7: 50, Resistor_THT:R_Axial_DIN0309_L9.0mm_D3.2mm_P12.70mm_Horizontal, F.Cu at (177.7, 128.4)
- added R7: 50, Resistor_THT:R_Axial_DIN0309_L9.0mm_D3.2mm_P12.70mm_Horizontal, F.Cu at (233.1, 147.8)
- moved D19 497.3 mm to (-33.7, 104.8), turned to 180 degrees
- moved C5 448.1 mm to (-5.30, 96.3), turned to -90 degrees
- moved C4 434.9 mm to (17.7, 96.3), turned to -90 degrees
- moved R27 409.6 mm to (190.1, -60.6)
- moved R28 409.6 mm to (190.1, -56.6)
- moved C6 404.1 mm to (26.4, 74.9), turned to 90 degrees
- moved R24 400.1 mm to (30.6, -7.30), turned to -90 degrees
- moved K4 400.0 mm to (212.4, 195.2), turned to 0 degrees
- moved R25 394.3 mm to (38.4, 7.26), turned to 90 degrees
- moved D6 383.4 mm to (249.2, 150.8), turned to 0 degrees
- moved R14 378.1 mm to (233.1, 189.3), turned to 0 degrees
- moved R23 370.1 mm to (233.1, 201.5), turned to 0 degrees
- moved J13 366.6 mm to (78.4, 83.0)
- moved J12 366.6 mm to (53.0, 47.5)
- moved R10 366.2 mm to (233.1, 173.2), turned to 0 degrees
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Other:
- board text removed: "120 VAC"
- board text removed: "3V3 GND_1 GPIO15 GPIO2 GPIO4 GPIO16 GPIO17 GPIO5 GPIO18 GPIO19 GPIO21 GPIO3 GPIO1 GPIO22 GPIO23"
- board text removed: "Bateria 12 VDC"
- board text removed: "Boton 1"
- board text removed: "Boton 2"
- board text removed: "Boton 3"
- board text removed: "Salida 1"
- board text removed: "Salida 2"
- board text removed: "Salida 3"
- board text removed: "Salida 4"
- board text removed: "Sensor IN"
- board text removed: "Sensor OUT"
- board text removed: "VIN1 GND_2 GPIO13 GPIO12 GPIO14 GPIO27 GPIO26 GPIO25 GPIO33 GPIO32 GPIO35 GPIO34 GPIO39 GPIO36 EN1"
