File: Panel_PCB/Panel_PCB.kicad_pcb (KiCad board)
At the start: 2 copper layers, 836.7 x 424.2 mm, 103 parts, among them J1 DC, J10 Relay 3, J11 Relay 4, J12 Terminal A, J13 Terminal B, J14 Boton D (4), J15 Control remoto, J2 Bateria, J3 Sensor IN, J4 Sensor OUT, J5 Boton A (1), J6 Boton B (2), J7 Boton C (3), J8 Relay 1, J9 Relay 2, K1 SANYOU_SRD_Form_C, K2 SANYOU_SRD_Form_C, K3 SANYOU_SRD_Form_C, K4 SANYOU_SRD_Form_C, K5 G6K-2P-Y, K6 G5LE-1-E, Q1 2N2222A, Q2 2N2222A, Q3 2N2222A, Q4 2N2222A, Q7 2N2222A, U1 TLP291, U10 LM1117T-3.3, U12 DS1307+, U13 LM311, U2 TLP291, U3 TLP291, U4 TLP291, U5 LM7805_TO220, U6 LM1117T-3.3, U7 LM7805_TO220, U8 LM7805_TO220, U9 LM1117T-3.3, Y1 Crystal

Commit message: Actualización de layout
Parts:
- removed the J9 at (190.4, 201.8)
- J1: value DC -> 12 VDC
- moved J8 194.8 mm to (68.6, 236.0), turned to 180 degrees
- moved U13 170.9 mm to (85.4, 15.8), turned to -90 degrees
- moved J9 168.4 mm to (92.0, 235.7), turned to 180 degrees
- moved K1 167.9 mm to (54.4, 201.2)
- moved D13 161.3 mm to (69.9, 21.3), turned to 90 degrees
- moved D12 151.7 mm to (93.3, 26.3), turned to -90 degrees
- moved J3 147.4 mm to (32.8, -91.8)
- moved J10 135.9 mm to (122.2, 235.7), turned to 180 degrees
- moved K2 135.8 mm to (82.6, 201.2)
- moved R18 134.5 mm to (87.5, 34.8), turned to 180 degrees
- moved D14 134.3 mm to (93.3, 11.1), turned to -90 degrees
- moved J4 131.1 mm to (48.7, -91.6)
- moved R26 112.9 mm to (88.2, 1.30), turned to 180 degrees
- moved C1 107.3 mm to (171.7, 6.30), turned to 180 degrees
- moved J5 106.6 mm to (73.9, -91.2)
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Connections:
- C1 pad 2: Net-(D10-A) -> Net-(D19-A)
- C3 pad 2: Net-(D10-A) -> Net-(D19-A)
- D2 pad 2: Net-(D10-A) -> Net-(D2-A)
- D8 pad 2: Net-(D10-A) -> Net-(D8-A)
- D9 pad 2: Net-(D10-A) -> Net-(D9-A)
- J15 pad 1: Net-(D10-A) -> Net-(D19-A)
- R16 pad 2: Net-(D10-K) -> Net-(D10-A)
- R17 pad 2: Net-(D9-K) -> Net-(D9-A)
- R21 pad 2: Net-(D10-A) -> Net-(D19-A)
- R26 pad 2: Net-(D10-A) -> Net-(D19-A)
- R27 pad 2: Net-(D8-K) -> Net-(D8-A)
- R28 pad 2: Net-(D2-K) -> Net-(D2-A)
- U13 pad 4: Net-(D10-A) -> Net-(D19-A)
- U5 pad 2: Net-(D10-A) -> Net-(D19-A)
- U6 pad 1: Net-(D10-A) -> Net-(D19-A)

Commit message: Organizando componentes en la PCB
Parts:
- removed the D4 at (178.0, 132.9)
- removed the R6 at (177.7, 137.1)
- removed the R7 at (177.7, 128.4)
- moved Q1 182.9 mm to (106.0, 74.8)
- moved U1 182.5 mm to (107.2, 60.2), turned to 90 degrees
- moved R4 180.7 mm to (105.8, 32.8), turned to -90 degrees
- moved R20 178.8 mm to (129.5, 47.6), turned to -90 degrees
- moved R1 175.3 mm to (96.2, 47.6), turned to -90 degrees
- moved R22 164.8 mm to (163.5, 48.0), turned to -90 degrees
- moved R6 162.7 mm to (141.4, 30.7), turned to -90 degrees
- moved Q2 161.3 mm to (136.1, 76.1)
- moved D3 161.1 mm to (96.2, 87.8), turned to 90 degrees
- moved U2 160.3 mm to (137.8, 59.8), turned to 90 degrees
- moved R11 159.2 mm to (115.0, 70.5), turned to 90 degrees
- moved R23 156.1 mm to (202.0, 48.5), turned to -90 degrees
- moved R8 152.0 mm to (170.6, 30.5), turned to -90 degrees
- moved R12 147.5 mm to (146.8, 61.6), turned to -90 degrees
- moved R10 145.9 mm to (209.9, 29.1), turned to -90 degrees
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
Commit message: Organizando componentes en la PCB
Parts:
- moved J3 123.2 mm to (84.6, -2.20)
- moved J4 123.2 mm to (97.5, -2.00)
- moved J15 123.2 mm to (192.5, -2.60)
- moved J5 123.2 mm to (122.7, -1.60)
- moved J6 123.2 mm to (136.9, -1.40)
- moved J14 123.2 mm to (164.8, -1.80)
- moved J7 123.2 mm to (150.9, -1.40)
- moved J1 55.6 mm to (-60.0, 94.0), turned to -90 degrees
- moved J2 53.2 mm to (-60.0, 79.4), turned to -90 degrees
- moved J8 26.6 mm to (90.0, 101.0)
- moved J9 26.5 mm to (130.0, 101.0)
- moved D10 26.4 mm to (68.4, 25.1)
- moved D12 26.4 mm to (8.18, 14.7)
- moved D14 26.4 mm to (8.18, -0.54)
- moved R16 26.4 mm to (67.7, -2.21)
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Routing:
- net Net-(D19-A): track 0.00 -> 778.4 mm, vias 0 -> 1
- net Net-(D12-A): track 0.00 -> 605.2 mm, vias 0 -> 1
- net Net-(J15-Pin_2): track 0.00 -> 309.0 mm, vias 0 -> 1
- net Net-(J14-Pin_1): track 0.00 -> 213.5 mm, vias 0 -> 2
- net Net-(J3-Pin_1): track 0.00 -> 201.7 mm, vias 0 -> 2
- net Net-(BT1--): track 0.00 -> 197.0 mm, vias 0 -> 3
- net Net-(D8-K): track 0.00 -> 184.9 mm, vias 0 -> 2
- net Net-(D2-K): track 0.00 -> 181.1 mm, vias 0 -> 2
- net Net-(J12-Pin_11): track 0.00 -> 175.5 mm, vias 0 -> 1
- net Net-(J15-Pin_3): track 0.00 -> 158.4 mm
- net Net-(J15-Pin_4): track 0.00 -> 152.9 mm, vias 0 -> 1
- net Net-(J13-Pin_8): track 0.00 -> 152.8 mm, vias 0 -> 1
- net Net-(J15-Pin_5): track 0.00 -> 146.1 mm
- net Net-(D10-K): track 0.00 -> 144.6 mm, vias 0 -> 1
- net Net-(D9-K): track 0.00 -> 141.2 mm, vias 0 -> 1
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Other:
- board size 836.7 x 424.2 mm -> 293.3 x 125 mm
- board text added: "+"
- board text added: "-"
- board text added: "12 VDC"
- board text added: "3V3 GND_1 GPIO15 GPIO2 GPIO4 GPIO16 GPIO17 GPIO5 GPIO18 GPIO19 GPIO21 GPIO3 GPIO1 GPIO22 GPIO23"
- board text added: "A"
- board text added: "B"
- board text added: "C"
- board text added: "D"
- board text added: "VIN1 GND_2 GPIO13 GPIO12 GPIO14 GPIO27 GPIO26 GPIO25 GPIO33 GPIO32 GPIO35 GPIO34 GPIO39 GPIO36 EN1"
- board text added: "bateria"
- board text added: "control remoto"
- board text added: "out 1"
- board text added: "out 2"
- board text added: "out 3"
- board text added: "out 4"
- board text added: "sensor in"
- board text added: "sensor out"

Commit message: Archivos de fabricacion
Parts:
- added h1: MountingHole_2.2mm_M2_DIN965_Pad, MountingHole:MountingHole_2.2mm_M2_DIN965_Pad, F.Cu at (-61.0, -10.1)
- added h1: MountingHole_2.2mm_M2_DIN965_Pad, MountingHole:MountingHole_2.2mm_M2_DIN965_Pad, F.Cu at (217.5, 105.5)
- added h1: MountingHole_2.2mm_M2_DIN965_Pad, MountingHole:MountingHole_2.2mm_M2_DIN965_Pad, F.Cu at (216.3, -7.30)
- added h1: MountingHole_2.2mm_M2_DIN965_Pad, MountingHole:MountingHole_2.2mm_M2_DIN965_Pad, F.Cu at (-60.7, 107.5)
- U1, U2, U3, U4: footprint Package_SO:SOIC-4_4.55x2.6mm_P1.27mm -> Package_DIP:DIP-4_W7.62mm
- moved R18 6.48 mm to (2.40, 24.1)
- moved R26 3.38 mm to (2.70, -6.50)
- moved R19 1.55 mm to (-10.9, 38.9)
- moved R25 1.24 mm to (35.1, 48.0)
- moved U6 0.42 mm to (24.9, 20.4)
- moved R2 0.40 mm to (49.5, 104.9)
Routing:
- net Net-(D12-A): track 605.2 -> 573.8 mm
- net Net-(D2-K): track 181.1 -> 159.6 mm
- net Net-(J13-Pin_3): track 89.0 -> 109.3 mm
- net Net-(D19-A): track 778.4 -> 797.9 mm, vias 1 -> 2
- net Net-(D8-K): track 184.9 -> 165.8 mm, vias 2 -> 1
- net Net-(K6-Pad3): track 60.9 -> 75.4 mm, vias 0 -> 1
- net Net-(J13-Pin_7): track 115.1 -> 102.1 mm, vias 1 -> 0
- net Net-(D10-K): track 144.6 -> 132.4 mm, vias 1 -> 0
- net Net-(J13-Pin_8): track 152.8 -> 142.1 mm, vias 1 -> 0
- net Net-(J3-Pin_1): track 201.7 -> 192.5 mm, vias 2 -> 1
- net Net-(J12-Pin_11): track 175.5 -> 184.3 mm, vias 1 -> 0
- net Net-(J13-Pin_5): track 126.6 -> 133.1 mm, vias 1 -> 2
- net Net-(R10-Pad2): track 14.2 -> 7.79 mm, vias 1 -> 0
- net Net-(J12-Pin_9): track 73.5 -> 67.1 mm
- net Net-(BT1--): track 197.0 -> 191.3 mm, vias 3 -> 2
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Other:
- board text added: "."
